File: BluetoothModule.sch (EAGLE design)
At the start: 25 parts, among them IC1 BL600, IC2 FT230XQ, J1 Autorun, J3 OTA, J6 USB

Commit message: tweaked USB connector footprint
Parts:
- J6: value USB -> (none); device freetronics-jon:USB-6PSMT -> freetronics-master-v1:M08STD
- J7: device freetronics-master-v1:M08STD -> freetronics-master-v1:M04PTH
- J8: value (none) -> USB; device freetronics-master-v1:M04PTH -> freetronics-master-v1:USB-MICROB
Connections:
- net +3V3: now also J7.3; no longer J8.3
- net ADC1: now also J6.6; no longer J7.6
- net ADC2: now also J6.5; no longer J7.5
- net ADC3: now also J6.4; no longer J7.4
- net ADC4: now also J6.3; no longer J7.3
- net ADC5: now also J6.2; no longer J7.2
- net ADC6: now also J6.1; no longer J7.1
- net GND: now also J7.4, J8.GND; no longer J6.FIX1, J6.FIX2, J6.GND, J6.PIN1, J6.PIN2, J6.TAB1, J6.TAB2, J8.4
- net N$11: now also J8.D-; no longer J6.D-
- net N$12: now also J8.D+; no longer J6.D+
- net N$5: now also J8.VBUS; no longer J6.VBUS
- net SIO0: now also J6.7; no longer J7.7
- net SIO25: now also J7.2; no longer J8.2
- net SIO29: now also J7.1; no longer J8.1
- net SIO30: now also J6.8; no longer J7.8
Changed lines of the file:
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@@
 <attribute name="VALUE2" value="FT230XQ"/>
 </part>
-<part name="J7" library="freetronics-master-v1" deviceset="M08" device="STD"/>
+<part name="J6" library="freetronics-master-v1" deviceset="M08" device="STD"/>
 <part name="+3V2" library="supply1" deviceset="+3V3" device="" value="+3.3V"/>
 <part name="C1" library="freetronics-master-v1" deviceset="CAP" device="0603" value="100nF">
@@
 <part name="J2" library="freetronics-master-v1" deviceset="M08" device="STD"/>
 <part name="J4" library="freetronics-master-v1" deviceset="M05" device="PTH"/>
-<part name="J8" library="freetronics-master-v1" deviceset="M04" device="PTH"/>
+<part name="J7" library="freetronics-master-v1" deviceset="M04" device="PTH"/>
 <part name="+3V3" library="supply1" deviceset="+3V3" device="" value="+3.3V"/>
 <part name="U$4" library="freetronics-luke" deviceset="GND" device=""/>
@@
 <attribute name="PACKAGE" value="0603"/>
 </part>
-<part name="J6" library="freetronics-jon" deviceset="USB-6P" device="SMT" value="USB"/>
 <part name="U$1" library="freetronics-luke" deviceset="GND" device=""/>
 <part name="C3" library="freetronics-master-v1" deviceset="CAP" device="0603" value="10nF">
@@
 <part name="+3V5" library="supply1" deviceset="+3V3" device="" value="+3.3V"/>
 <part name="U$11" library="freetronics-luke" deviceset="GND" device=""/>
+<part name="J8" library="freetronics-master-v1" deviceset="USB" device="-MICROB" value="USB"/>
 </parts>
 <sheets>
@@
 <attribute name="PACKAGE" x="160.02" y="114.3" size="1.27" layer="96"/>
 </instance>
-<instance part="J7" gate="G$1" x="345.44" y="93.98" smashed="yes" rot="R180">
+<instance part="J6" gate="G$1" x="345.44" y="93.98" smashed="yes" rot="R180">
 <attribute name="VALUE" x="350.52" y="106.68" size="1.778" layer="96" rot="R180"/>
 <attribute name="NAME" x="344.17" y="104.648" size="1.27" layer="95"/>
@@
 <attribute name="NAME" x="316.23" y="117.348" size="1.27" layer="95"/>
 </instance>
-<instance part="J8" gate="G$1" x="317.5" y="88.9" smashed="yes" rot="R180">
+<instance part="J7" gate="G$1" x="317.5" y="88.9" smashed="yes" rot="R180">
 <attribute name="VALUE" x="322.58" y="96.52" size="1.778" layer="96" rot="R180"/>
 <attribute name="NAME" x="316.23" y="94.488" size="1.27" layer="95"/>
@@
 <attribute name="VALUE" x="208.28" y="63.5" size="1.27" layer="96"/>
 </instance>
-<instance part="J6" gate="G$1" x="40.64" y="96.52" smashed="yes" rot="R180">
-<attribute name="NAME" x="35.56" y="119.38" size="1.27" layer="95"/>
-<attribute name="VALUE" x="35.56" y="116.84" size="1.27" layer="96"/>
-</instance>
-<instance part="U$1" gate="G$1" x="50.8" y="73.66"/>
+<instance part="U$1" gate="G$1" x="50.8" y="81.28"/>
 <instance part="C3" gate="G$1" x="58.42" y="91.44" smashed="yes" rot="R180">
 <attribute name="NAME" x="63.5" y="91.44" size="1.27" layer="95"/>
@@
 </instance>
 <instance part="U$11" gate="G$1" x="340.36" y="127" rot="MR0"/>
+<instance part="J8" gate="G$1" x="45.72" y="93.98" rot="MR0"/>
 </instances>
 <busses>
@@
 </segment>
 <segment>
-<pinref part="J8" gate="G$1" pin="4"/>
+<pinref part="J7" gate="G$1" pin="4"/>
 <wire x1="312.42" y1="83.82" x2="309.88" y2="83.82" width="0.1524" layer="91"/>
 <pinref part="U$4" gate="G$1" pin="GND"/>
@@
 </segment>
 <segment>
-<pinref part="J6" gate="G$1" pin="FIX1"/>
-<wire x1="38.1" y1="109.22" x2="38.1" y2="114.3" width="0.1524" layer="91"/>
-<wire x1="38.1" y1="114.3" x2="40.64" y2="114.3" width="0.1524" layer="91"/>
-<pinref part="J6" gate="G$1" pin="TAB1"/>
-<wire x1="40.64" y1="114.3" x2="40.64" y2="109.22" width="0.1524" layer="91"/>
-<wire x1="40.64" y1="114.3" x2="50.8" y2="114.3" width="0.1524" layer="91"/>
-<wire x1="50.8" y1="114.3" x2="50.8" y2="104.14" width="0.1524" layer="91"/>
-<pinref part="J6" gate="G$1" pin="PIN1"/>
-<wire x1="45.72" y1="104.14" x2="50.8" y2="104.14" width="0.1524" layer="91"/>
-<wire x1="50.8" y1="104.14" x2="50.8" y2="91.44" width="0.1524" layer="91"/>
-<pinref part="J6" gate="G$1" pin="GND"/>
-<wire x1="45.72" y1="91.44" x2="50.8" y2="91.44" width="0.1524" layer="91"/>
-<wire x1="50.8" y1="91.44" x2="50.8" y2="88.9" width="0.1524" layer="91"/>
-<pinref part="J6" gate="G$1" pin="PIN2"/>
-<wire x1="45.72" y1="88.9" x2="50.8" y2="88.9" width="0.1524" layer="91"/>
-<wire x1="50.8" y1="88.9" x2="50.8" y2="78.74" width="0.1524" layer="91"/>
-<wire x1="50.8" y1="78.74" x2="40.64" y2="78.74" width="0.1524" layer="91"/>
-<pinref part="J6" gate="G$1" pin="TAB2"/>
-<pinref part="J6" gate="G$1" pin="FIX2"/>
-<wire x1="40.64" y1="83.82" x2="40.64" y2="78.74" width="0.1524" layer="91"/>
-<wire x1="40.64" y1="78.74" x2="38.1" y2="78.74" width="0.1524" layer="91"/>
-<wire x1="38.1" y1="78.74" x2="38.1" y2="83.82" width="0.1524" layer="91"/>
-<pinref part="U$1" gate="G$1" pin="GND"/>
-<wire x1="50.8" y1="76.2" x2="50.8" y2="78.74" width="0.1524" layer="91"/>
-<junction x="40.64" y="78.74"/>
-<junction x="50.8" y="91.44"/>
-<junction x="50.8" y="88.9"/>
-<junction x="40.64" y="114.3"/>
-<junction x="50.8" y="104.14"/>
-<junction x="50.8" y="78.74"/>
-</segment>
-<segment>
 <pinref part="C3" gate="G$1" pin="1"/>
 <pinref part="U$5" gate="G$1" pin="GND"/>
@@
 <pinref part="U$11" gate="G$1" pin="GND"/>
 <wire x1="340.36" y1="129.54" x2="340.36" y2="132.08" width="0.1524" layer="91"/>
+</segment>
+<segment>
+<pinref part="J8" gate="G$1" pin="GND"/>
+<wire x1="48.26" y1="93.98" x2="50.8" y2="93.98" width="0.1524" layer="91"/>
+<wire x1="50.8" y1="93.98" x2="50.8" y2="83.82" width="0.1524" layer="91"/>
+<pinref part="U$1" gate="G$1" pin="GND"/>
 </segment>
 </net>
@@
 </segment>
 <segment>
-<pinref part="J8" gate="G$1" pin="3"/>
+<pinref part="J7" gate="G$1" pin="3"/>
 <pinref part="+3V3" gate="G$1" pin="+3V3"/>
 <wire x1="312.42" y1="86.36" x2="309.88" y2="86.36" width="0.1524" layer="91"/>
@@
 </segment>
 <segment>
-<pinref part="J7" gate="G$1" pin="7"/>
+<pinref part="J6" gate="G$1" pin="7"/>
 <wire x1="340.36" y1="86.36" x2="327.66" y2="86.36" width="0.1524" layer="91"/>
 <label x="330.2" y="86.614" size="1.27" layer="95"/>
@@
 </segment>
 <segment>
-<pinref part="J7" gate="G$1" pin="6"/>
+<pinref part="J6" gate="G$1" pin="6"/>
 <wire x1="340.36" y1="88.9" x2="327.66" y2="88.9" width="0.1524" layer="91"/>
 <label x="330.2" y="89.154" size="1.27" layer="95"/>
@@
 </segment>
 <segment>
-<pinref part="J7" gate="G$1" pin="5"/>
+<pinref part="J6" gate="G$1" pin="5"/>
 <wire x1="340.36" y1="91.44" x2="327.66" y2="91.44" width="0.1524" layer="91"/>
 <label x="330.2" y="91.694" size="1.27" layer="95"/>
@@
 </segment>
 <segment>
-<pinref part="J7" gate="G$1" pin="4"/>
+<pinref part="J6" gate="G$1" pin="4"/>
 <wire x1="340.36" y1="93.98" x2="327.66" y2="93.98" width="0.1524" layer="91"/>
 <label x="330.2" y="94.234" size="1.27" layer="95"/>
@@
 </segment>
 <segment>
-<pinref part="J7" gate="G$1" pin="3"/>
+<pinref part="J6" gate="G$1" pin="3"/>
 <wire x1="340.36" y1="96.52" x2="327.66" y2="96.52" width="0.1524" layer="91"/>
 <label x="330.2" y="96.774" size="1.27" layer="95"/>
@@
 </segment>
 <segment>
-<pinref part="J7" gate="G$1" pin="2"/>
+<pinref part="J6" gate="G$1" pin="2"/>
 <wire x1="340.36" y1="99.06" x2="327.66" y2="99.06" width="0.1524" layer="91"/>
 <label x="330.2" y="99.314" size="1.27" layer="95"/>
@@
 </segment>
 <segment>
-<pinref part="J7" gate="G$1" pin="1"/>
+<pinref part="J6" gate="G$1" pin="1"/>
 <wire x1="340.36" y1="101.6" x2="327.66" y2="101.6" width="0.1524" layer="91"/>
 <label x="330.2" y="101.854" size="1.27" layer="95"/>
@@
 </segment>
 <segment>
-<pinref part="J7" gate="G$1" pin="8"/>
+<pinref part="J6" gate="G$1" pin="8"/>
 <wire x1="340.36" y1="83.82" x2="327.66" y2="83.82" width="0.1524" layer="91"/>
 <label x="330.2" y="84.074" size="1.27" layer="95"/>
@@
 </segment>
 <segment>
-<pinref part="J8" gate="G$1" pin="1"/>
+<pinref part="J7" gate="G$1" pin="1"/>
 <wire x1="312.42" y1="91.44" x2="299.72" y2="91.44" width="0.1524" layer="91"/>
 <label x="302.26" y="91.694" size="1.27" layer="95"/>
@@
 </segment>
 <segment>
-<pinref part="J8" gate="G$1" pin="2"/>
+<pinref part="J7" gate="G$1" pin="2"/>
 <wire x1="312.42" y1="88.9" x2="299.72" y2="88.9" width="0.1524" layer="91"/>
 <label x="302.26" y="89.154" size="1.27" layer="95"/>
@@
 <net name="N$5" class="0">
 <segment>
-<pinref part="J6" gate="G$1" pin="VBUS"/>
-<wire x1="45.72" y1="101.6" x2="55.88" y2="101.6" width="0.1524" layer="91"/>
+<wire x1="48.26" y1="101.6" x2="55.88" y2="101.6" width="0.1524" layer="91"/>
 <wire x1="55.88" y1="101.6" x2="58.42" y2="104.14" width="0.1524" layer="91"/>
 <pinref part="C3" gate="G$1" pin="2"/>
@@
 <wire x1="58.42" y1="104.14" x2="60.96" y2="104.14" width="0.1524" layer="91"/>
 <junction x="58.42" y="104.14"/>
+<pinref part="J8" gate="G$1" pin="VBUS"/>
 </segment>
 </net>
@@
 <net name="N$11" class="0">
 <segment>
-<pinref part="J6" gate="G$1" pin="D-"/>
-<wire x1="45.72" y1="99.06" x2="73.66" y2="99.06" width="0.1524" layer="91"/>
+<wire x1="48.26" y1="99.06" x2="73.66" y2="99.06" width="0.1524" layer="91"/>
 <pinref part="C4" gate="G$1" pin="2"/>
 <wire x1="73.66" y1="93.98" x2="73.66" y2="99.06" width="0.1524" layer="91"/>
@@
 <wire x1="139.7" y1="99.06" x2="73.66" y2="99.06" width="0.1524" layer="91"/>
 <junction x="73.66" y="99.06"/>
+<pinref part="J8" gate="G$1" pin="D-"/>
 </segment>
 </net>
 <net name="N$12" class="0">
 <segment>
-<pinref part="J6" gate="G$1" pin="D+"/>
-<wire x1="45.72" y1="96.52" x2="88.9" y2="96.52" width="0.1524" layer="91"/>
+<wire x1="48.26" y1="96.52" x2="88.9" y2="96.52" width="0.1524" layer="91"/>
 <pinref part="C5" gate="G$1" pin="2"/>
 <wire x1="88.9" y1="93.98" x2="88.9" y2="96.52" width="0.1524" layer="91"/>
@@
 <wire x1="129.54" y1="96.52" x2="88.9" y2="96.52" width="0.1524" layer="91"/>
 <junction x="88.9" y="96.52"/>
-</segment>
-</net>
+<pinref part="J8" gate="G$1" pin="D+"/>
+</segment>
+</net>
